Commit message: add basefootprint joint & link

File: description/robot_core.xacro (robot description, xacro)
@@ -19,4 +19,13 @@
     <!-- BASE LINK -->
     <link name="base_link">
+    </link>
+    <!-- BASE FOOTPRINT LINK -->
+    <joint name="base_footprint_link" type="fixed">
+        <parent link="base_link">
+            <child link="base_footprint"/>
+            <origin xyz="0 0 0" rpy="0 0 0"/>
+        </parent>
+    </joint>
+    <link name="base_footprint">
     </link>
     <!-- CHASSIS LINK -->

Commit message: fix footprint link

File: description/robot_core.xacro (robot description, xacro)
@@ -21,9 +21,8 @@
     </link>
     <!-- BASE FOOTPRINT LINK -->
-    <joint name="base_footprint_link" type="fixed">
-        <parent link="base_link">
-            <child link="base_footprint"/>
-            <origin xyz="0 0 0" rpy="0 0 0"/>
-        </parent>
+    <joint name="base_footprint_joint" type="fixed">
+        <parent link="base_link"/>
+        <child link="base_footprint"/>
+        <origin xyz="0 0 0" rpy="0 0 0"/>
     </joint>
     <link name="base_footprint">
